Commit message: add limit to joint_1, reduce the odds of flipping all over

File: isaac-sim2real/tm5s.urdf (robot description, URDF)
Before this commit: robot tm5s, 9 links, 8 joints
Joints:
- joint joint_1: limit lower=-6.283185307179586 upper=6.283185307179586 effort=170 velocity=0.73 -> lower=-1.0 upper=6.283185307179586 effort=170 velocity=0.73

Commit message: Can avoid most of the weird plans for now

File: isaac-sim2real/tm5s.urdf (robot description, URDF)
Before this commit: robot tm5s, 9 links, 8 joints
Joints:
- joint joint_3: limit lower=-2.7576202181510405 upper=2.7576202181510405 effort=170 velocity=0.73 -> lower=-0.8 upper=2.7576202181510405 effort=170 velocity=0.73
- joint joint_5: limit lower=-6.283185307179586 upper=6.283185307179586 effort=45 velocity=0.78 -> lower=-6.283185307179586 upper=2.5 effort=45 velocity=0.78
- joint joint_6: limit lower=-6.283185307179586 upper=6.283185307179586 effort=45 velocity=1.56 -> lower=-1.5 upper=6.283185307179586 effort=45 velocity=1.56

Commit message: nice settings

File: isaac-sim2real/tm5s.urdf (robot description, URDF)
Before this commit: robot tm5s, 9 links, 8 joints
Joints:
- joint joint_1: limit lower=-1.0 upper=6.283185307179586 effort=170 velocity=0.73 -> lower=-1.0 upper=3.14 effort=170 velocity=0.73
- joint joint_4: limit lower=-6.283185307179586 upper=6.283185307179586 effort=45 velocity=0.78 -> lower=-1.5 upper=4.04 effort=45 velocity=0.78

Commit message: 04011426

File: isaac-sim2real/tm5s.urdf (robot description, URDF)
Before this commit: robot tm5s, 9 links, 8 joints
Joints:
- joint joint_1: limit lower=-1.0 upper=3.14 effort=170 velocity=0.73 -> lower=-6.283185307179586 upper=6.283185307179586 effort=170 velocity=3.6651914291880923
- joint joint_2: limit lower=-6.283185307179586 upper=6.283185307179586 effort=170 velocity=0.73 -> lower=-6.283185307179586 upper=6.283185307179586 effort=170 velocity=3.6651914291880923
- joint joint_3: limit lower=-0.8 upper=2.7576202181510405 effort=170 velocity=0.73 -> lower=-2.7576202181510405 upper=2.7576202181510405 effort=170 velocity=3.6651914291880923
- joint joint_4: limit lower=-1.5 upper=4.04 effort=45 velocity=0.78 -> lower=-6.283185307179586 upper=6.283185307179586 effort=45 velocity=3.9269908169872414
- joint joint_5: limit lower=-6.283185307179586 upper=2.5 effort=45 velocity=0.78 -> lower=-6.283185307179586 upper=6.283185307179586 effort=45 velocity=3.9269908169872414
- joint joint_6: limit lower=-1.5 upper=6.283185307179586 effort=45 velocity=1.56 -> lower=-6.283185307179586 upper=6.283185307179586 effort=45 velocity=7.853981633974483

Commit message: temp 0402

File: isaac-sim2real/tm5s.urdf (robot description, URDF)
Before this commit: robot tm5s, 9 links, 8 joints
Joints:
- joint joint_1: limit lower=-6.283185307179586 upper=6.283185307179586 effort=170 velocity=3.6651914291880923 -> lower=-1.0 upper=3.14 effort=170 velocity=0.73
- joint joint_2: limit lower=-6.283185307179586 upper=6.283185307179586 effort=170 velocity=3.6651914291880923 -> lower=-5.283185307179586 upper=5.283185307179586 effort=170 velocity=0.73
- joint joint_3: limit lower=-2.7576202181510405 upper=2.7576202181510405 effort=170 velocity=3.6651914291880923 -> lower=-0.8 upper=2.7576202181510405 effort=170 velocity=0.73
- joint joint_4: limit lower=-6.283185307179586 upper=6.283185307179586 effort=45 velocity=3.9269908169872414 -> lower=-1.5 upper=4.04 effort=45 velocity=0.78
- joint joint_5: limit lower=-6.283185307179586 upper=6.283185307179586 effort=45 velocity=3.9269908169872414 -> lower=-6.283185307179586 upper=2.5 effort=45 velocity=0.78
- joint joint_6: limit lower=-6.283185307179586 upper=6.283185307179586 effort=45 velocity=7.853981633974483 -> lower=-1.5 upper=6.283185307179586 effort=45 velocity=1.56

Commit message: 04091354

File: isaac-sim2real/tm5s.urdf (robot description, URDF)
Before this commit: robot tm5s, 9 links, 8 joints
Joints:
- joint joint_2: limit lower=-5.283185307179586 upper=5.283185307179586 effort=170 velocity=0.73 -> lower=-6.283185307179586 upper=6.283185307179586 effort=170 velocity=0.73
